Commit message: Fix: Resolve OGRE Material warnings on launch (#28)
* fix: Replace OGRE specific colors with modern Gazebo color definitions.

* fix: Switch URDF files to colors defined in the materials.xacro file.

* feat: Add dark_gray color to previously uncolored sensor components.

File: ora_description/description/anteater_core.xacro (robot description, xacro)
@@ -41,5 +41,5 @@
   </link>
   <gazebo reference="chassis_link">
-    <material>Gazebo/White</material>
+    <material name="white"/>
   </gazebo>
 </robot>

File: ora_description/description/caster.xacro (robot description, xacro)
@@ -13,5 +13,5 @@
           <cylinder radius="${front_caster_radius}" length="${front_caster_width}"/>
         </geometry>
-        <material name="gray"/>
+        <material name="black"/>
       </visual>
       <collision>
@@ -31,9 +31,9 @@
     </joint>
     <gazebo reference="${prefix}_front_caster_link">
-      <material>Gazebo/Black</material>
+      <material name="black"/>
       <!-- Frictionless-ish -->
       <!-- Stops the robot from jumping around -->
-      <mu1 value="0.001"/>
-      <mu2 value="0.001"/>
+      <mu1>0.001</mu1>
+      <mu2>0.001</mu2>
     </gazebo>
   </xacro:macro>
@@ -48,5 +48,5 @@
           <cylinder radius="${back_caster_radius}" length="${back_caster_width}"/>
         </geometry>
-        <material name="gray"/>
+        <material name="black"/>
       </visual>
       <collision>
@@ -66,9 +66,9 @@
     </joint>
     <gazebo reference="${prefix}_back_caster_link">
-      <material>Gazebo/Black</material>
+      <material name="black"/>
       <!-- Frictionless-ish -->
       <!-- Stops the robot from jumping around -->
-      <mu1 value="0.001"/>
-      <mu2 value="0.001"/>
+      <mu1>0.001</mu1>
+      <mu2>0.001</mu2>
     </gazebo>
   </xacro:macro>

File: ora_description/description/wheel.xacro (robot description, xacro)
@@ -27,5 +27,5 @@
     </link>
     <gazebo reference="${prefix}_wheel_link">
-      <material>Gazebo/Black</material>
+      <material name="black"/>
     </gazebo>
   </xacro:macro>
